Commit message: Update meshes and urdf files

File: urdf/robotiq_140_gripper.urdf (robot description, URDF)
Before this commit: robot robotiq_140_gripper, 1 links, 0 joints
Links:
- removed link base_link
- added link world

File: urdf/robotiq_140_gripper.urdf.xacro (robot description, xacro)
@@ -210,5 +210,5 @@
   </xacro:macro>
   <xacro:include filename="$(find aist_robotiq
-			   )/urdf/robotiq_arg2f.urdf.xacro"/>
+			   )/urdf/robotiq_arg2f.xacro"/>
   <xacro:macro name="finger_joint" params="prefix">
     <joint name="${prefix}finger_joint" type="revolute">
@@ -235,12 +235,12 @@
   <!-- Initialization of all joints and links -->
   <xacro:macro name="robotiq_140_gripper" params="prefix parent *origin">
-    <joint name="${prefix}robotiq_140_base_joint" type="fixed">
+    <joint name="${prefix}base_joint" type="fixed">
       <parent link="${parent}"/>
-      <child  link="${prefix}robotiq_140_base_link"/>
+      <child  link="${prefix}base_link"/>
       <xacro:insert_block name="origin"/>
     </joint>
-    <link  name="${prefix}robotiq_140_base_link"/>
+    <link  name="${prefix}base_link"/>
     <joint name="${prefix}robotiq_arg2f_base_joint" type="fixed">
-      <parent link="${prefix}robotiq_140_base_link"/>
+      <parent link="${prefix}base_link"/>
       <child  link="${prefix}robotiq_arg2f_base_link"/>
       <origin xyz="0 0 0" rpy="${pi} ${-pi/2} 0"/>

File: urdf/robotiq_85_gripper.urdf (robot description, URDF)
Before this commit: robot robotiq_85_gripper, 1 links, 0 joints
Links:
- removed link base_link
- added link world

File: urdf/robotiq_85_gripper.urdf.xacro (robot description, xacro)
@@ -201,5 +201,5 @@
   </xacro:macro>
   <xacro:include filename="$(find aist_robotiq
-			   )/urdf/robotiq_arg2f.urdf.xacro"/>
+			   )/urdf/robotiq_arg2f.xacro"/>
   <xacro:macro name="finger_joint" params="prefix">
     <joint name="${prefix}finger_joint" type="revolute">
@@ -226,12 +226,12 @@
   <!-- Initialization of all joints and links -->
   <xacro:macro name="robotiq_85_gripper" params="prefix parent *origin">
-    <joint name="${prefix}robotiq_85_base_joint" type="fixed">
+    <joint name="${prefix}base_joint" type="fixed">
       <parent link="${parent}"/>
-      <child  link="${prefix}robotiq_85_base_link"/>
+      <child  link="${prefix}base_link"/>
       <xacro:insert_block name="origin"/>
     </joint>
-    <link  name="${prefix}robotiq_85_base_link"/>
+    <link  name="${prefix}base_link"/>
     <joint name="${prefix}robotiq_arg2f_base_joint" type="fixed">
-      <parent link="${prefix}robotiq_85_base_link"/>
+      <parent link="${prefix}base_link"/>
       <child  link="${prefix}robotiq_arg2f_base_link"/>
       <origin xyz="0 0 0" rpy="${pi} ${-pi/2} 0"/>

File: urdf/robotiq_arg2f_coupling.urdf (robot description, URDF)
Before this commit: robot robotiq_arg2f_coupling, 1 links, 0 joints
Links:
- removed link base_link
- added link world

File: urdf/robotiq_arg2f_coupling.urdf.xacro (robot description, xacro)
@@ -4,5 +4,5 @@
     <xacro:property name="coupling_radius" value="0.0375"/>
     <xacro:property name="coupling_length" value="0.0169"/>
-    <link name="${prefix}robotiq_arg2f_coupling_link">
+    <link name="${prefix}base_link">
       <inertial>
         <origin xyz="8.625E-08 -4.6583E-06 0.03145" rpy="0 0 0" />
@@ -31,17 +31,17 @@
       </collision>
     </link>
-    <gazebo reference="${prefix}robotiq_arg2f_coupling_link">
+    <gazebo reference="${prefix}base_link">
       <material>Gazebo/Black</material>
     </gazebo>
     <!-- Add the force sensor in front of the gripper. -->
-    <joint name="${prefix}robotiq_arg2f_coupling_joint" type="fixed">
+    <joint name="${prefix}base_joint" type="fixed">
       <parent link="${parent}"/>
-      <child  link="${prefix}robotiq_arg2f_coupling_link"/>
+      <child  link="${prefix}base_link"/>
       <xacro:insert_block name="origin"/>
     </joint>
-    <link name="${prefix}robotiq_arg2f_coupling_flange_link"/>
-    <joint name="${prefix}robotiq_arg2f_coupling_flange_joint" type="fixed">
-      <parent link="${prefix}robotiq_arg2f_coupling_link"/>
-      <child  link="${prefix}robotiq_arg2f_coupling_flange_link"/>
+    <link name="${prefix}flange_link"/>
+    <joint name="${prefix}flange_joint" type="fixed">
+      <parent link="${prefix}base_link"/>
+      <child  link="${prefix}flange_link"/>
       <origin xyz="${coupling_length} 0 0" rpy="0 0 0"/>
     </joint>

File: urdf/robotiq_hande_gripper.urdf (robot description, URDF)
Before this commit: robot robotiq_hande, 1 links, 0 joints
Links:
- removed link base_link
- added link world

File: urdf/robotiq_hande_gripper.urdf.xacro (robot description, xacro)
@@ -1,111 +1,135 @@
 <?xml version="1.0"?>
 <robot xmlns:xacro="http://ros.org/wiki/xacro">
-  <xacro:macro name="robotiq_hande_gripper"  params="prefix parent *origin">
-    <joint name="${prefix}robotiq_hande_base_joint" type="fixed">
+  <!--
+  Author: Cristian Beltran
+-->
+  <xacro:macro name="robotiq_hande_gripper" params="prefix parent *origin">
+    <xacro:include filename="$(find aist_robotiq
+			     )/urdf/robotiq_arg2f_transmission.xacro"/>
+    <xacro:robotiq_arg2f_transmission prefix="${prefix}"/>
+    <joint name="${prefix}base_joint" type="fixed">
       <parent link="${parent}"/>
-      <child link="${prefix}robotiq_hande_base_link"/>
+      <child link="${prefix}base_link"/>
       <xacro:insert_block name="origin"/>
     </joint>
-    <link name="${prefix}robotiq_hande_base_link">
+    <link name="${prefix}base_link"/>
+    <joint name="${prefix}hande_joint" type="fixed">
+      <parent link="${prefix}base_link"/>
+      <child link="${prefix}hande_link"/>
+      <origin xyz="0 0 0" rpy="${pi/2} 0 ${pi/2}"/>
+    </joint>
+    <link name="${prefix}hande_link">
       <inertial>
-        <origin xyz="0 0 0.04607" rpy="${pi/2} 0 ${pi/2}" />
-        <mass value="0.86387" />
-        <inertia ixx="1017560E-9" ixy="0" ixz="2235E-9" iyy="1028041E-9" iyz="0" izz="489810E-9" />
+        <origin rpy="0 0 0" xyz="0 0 0.04607"/>
+        <mass value="0.86387"/>
+        <inertia ixx="1017560E-9" ixy="0" ixz="2235E-9" iyy="1028041E-9" iyz="0" izz="489810E-9"/>
       </inertial>
       <visual>
-        <origin xyz="0 0 0" rpy="${pi/2} 0 ${pi/2}" />
+        <origin rpy="0 0 0" xyz="0 0 0"/>
         <geometry>
-          <mesh filename="package://aist_robotiq/meshes/visual/hand-e.dae" scale="0.001 0.001 0.001"/>
+          <mesh filename="package://aist_robotiq/meshes/visual/robotiq_hande.dae" scale="1.0 1.0 1.0"/>
         </geometry>
-        <material name="Gazebo/Black">
-          <color rgba="0.1 0.1 0.1 1" />
+        <material name="Dark">
+          <color rgba=".1 0.1 0.1 1.0"/>
         </material>
       </visual>
       <collision>
-        <origin xyz="0 0 0" rpy="${pi/2} 0 ${pi/2}" />
+        <origin rpy="0 0 0" xyz="0 0 0"/>
         <geometry>
-          <mesh filename="package://aist_robotiq/meshes/visual/hand-e.dae" scale="0.001 0.001 0.001"/>
+          <mesh filename="package://aist_robotiq/meshes/collision/robotiq_hande-collision.dae" scale="1.0 1.0 1.0"/>
         </geometry>
       </collision>
     </link>
-    <gazebo reference="${prefix}robotiq_hande_base_link">
-      <material>Gazebo/Black</material>
-      <selfCollide>True</selfCollide>
-    </gazebo>
-    <link name="${prefix}robotiq_hande_left_finger">
+    <link name="${prefix}left_finger">
       <inertial>
-        <origin xyz="0.02262 -0.00759 0.00738" rpy="${pi/2} 0 ${pi/2}"/>
+        <origin rpy="0 0 0" xyz="0.02262 -0.00759 0.00738"/>
         <mass value="0.03804"/>
         <inertia ixx="13567E-9" ixy="1849E-9" ixz="3622E-9" iyy="15784E-9" iyz="3616E-9" izz="7478E-9"/>
       </inertial>
       <visual>
-        <origin xyz="0 0 0" rpy="${pi/2} 0 ${pi/2}"/>
+        <origin rpy="0 0 0" xyz="0 0 0"/>
         <geometry>
-          <mesh filename="package://aist_robotiq/meshes/visual/hand-e_finger_1.dae" scale="0.001 0.001 0.001"/>
+          <mesh filename="package://aist_robotiq/meshes/visual/robotiq_hande_finger_1.dae" scale="1.0 1.0 1.0"/>
         </geometry>
-        <material name="Gazebo/White">
-          <color rgba="1 1 1 1"/>
+        <material name="DarkGray">
+          <color rgba=".4 0.4 0.4 1.0"/>
         </material>
       </visual>
       <collision>
-        <origin xyz="0 0 0" rpy="${pi/2} 0 ${pi/2}"/>
+        <origin rpy="0 0 0" xyz="0 0 0"/>
         <geometry>
-          <mesh filename="package://aist_robotiq/meshes/visual/hand-e_finger_1.dae" scale="0.001 0.001 0.001"/>
+          <mesh filename="package://aist_robotiq/meshes/collision/robotiq_hande_finger_1-collision.dae" scale="1.0 1.0 1.0"/>
         </geometry>
       </collision>
     </link>
-    <gazebo reference="${prefix}robotiq_hande_left_finger">
-      <material>Gazebo/White</material>
-      <selfCollide>True</selfCollide>
-    </gazebo>
-    <link name="${prefix}robotiq_hande_right_finger">
+    <link name="${prefix}right_finger">
       <inertial>
-        <origin xyz="-0.02262 0.00759 0.00738" rpy="${pi/2} 0 ${pi/2}"/>
+        <origin rpy="0 0 0" xyz="-0.02262 0.00759 0.00738"/>
         <mass value="0.03804"/>
         <inertia ixx="13567E-9" ixy="1849E-9" ixz="-3622E-9" iyy="15784E-9" iyz="-3616E-9" izz="7478E-9"/>
       </inertial>
       <visual>
-        <origin xyz="0 0 0" rpy="${pi/2} 0 ${pi/2}"/>
+        <origin rpy="0 0 0" xyz="0 0 0"/>
         <geometry>
-          <mesh filename="package://aist_robotiq/meshes/visual/hand-e_finger_2.dae" scale="0.001 0.001 0.001"/>
+          <mesh filename="package://aist_robotiq/meshes/visual/robotiq_hande_finger_2.dae" scale="1.0 1.0 1.0"/>
         </geometry>
-        <material name="Gazebo/White">
-          <color rgba="1 1 1 1"/>
+        <material name="DarkGray">
+          <color rgba=".4 0.4 0.4 1.0"/>
         </material>
       </visual>
       <collision>
-        <origin xyz="0 0 0" rpy="${pi/2} 0 ${pi/2}"/>
+        <origin rpy="0 0 0" xyz="0 0 0"/>
         <geometry>
-          <mesh filename="package://aist_robotiq/meshes/visual/hand-e_finger_2.dae" scale="0.001 0.001 0.001"/>
+          <mesh filename="package://aist_robotiq/meshes/collision/robotiq_hande_finger_2-collision.dae" scale="1.0 1.0 1.0"/>
         </geometry>
       </collision>
     </link>
-    <gazebo reference="${prefix}robotiq_hande_right_finger">
-      <material>Gazebo/White</material>
-      <selfCollide>True</selfCollide>
+    <gazebo reference="${prefix}hande_link">
+      <material>Gazebo/FlatBlack</material>
+    </gazebo>
+    <gazebo reference="${prefix}right_finger">
+      <material>Gazebo/Grey</material>
+    </gazebo>
+    <gazebo reference="${prefix}left_finger">
+      <material>Gazebo/Grey</material>
     </gazebo>
     <joint name="${prefix}finger_joint" type="prismatic">
-      <origin xyz="0.099 0 0" rpy="0 0 0"/>
-      <parent link="${prefix}robotiq_hande_base_link"/>
-      <child link="${prefix}robotiq_hande_left_finger"/>
-      <axis xyz="0 -1 0"/>
+      <origin rpy="0 0 0" xyz="0 0 0.099"/>
+      <parent link="${prefix}hande_link"/>
+      <child link="${prefix}left_finger"/>
+      <axis xyz="-1 0 0"/>
       <limit effort="130" lower="0" upper="0.025" velocity="0.15"/>
     </joint>
-    <joint name="${prefix}robotiq_hande_base_to_right_finger" type="prismatic">
-      <origin xyz="0.099 0 0" rpy="0 0 0"/>
-      <parent link="${prefix}robotiq_hande_base_link"/>
-      <child link="${prefix}robotiq_hande_right_finger"/>
-      <axis xyz="0 1 0"/>
+    <joint name="${prefix}right_finger_joint" type="prismatic">
+      <origin rpy="0 0 0" xyz="0 0 0.099"/>
+      <parent link="${prefix}hande_link"/>
+      <child link="${prefix}right_finger"/>
+      <axis xyz="1 0 0"/>
       <limit effort="130" lower="0" upper="0.025" velocity="0.15"/>
       <mimic joint="${prefix}finger_joint" multiplier="1" offset="0"/>
     </joint>
-    <xacro:include filename="$(find aist_robotiq
-			     )/urdf/robotiq_arg2f_transmission.xacro"/>
-    <xacro:robotiq_arg2f_transmission prefix="${prefix}"/>
+    <!-- Improve grasping physics -->
+    <gazebo reference="${prefix}left_finger">
+      <kp>1000000.0</kp>
+      <kd>1.0</kd>
+      <mu1>1.0</mu1>
+      <mu2>1.0</mu2>
+      <minDepth>0.001</minDepth>
+    </gazebo>
+    <gazebo reference="${prefix}right_finger">
+      <kp>1000000.0</kp>
+      <kd>1.0</kd>
+      <mu1>1.0</mu1>
+      <mu2>1.0</mu2>
+      <minDepth>0.001</minDepth>
+    </gazebo>
+    <!-- Mimic joints -->
     <gazebo>
       <plugin filename="libgazebo_mimic_joint_plugin.so"
 	      name="${prefix}mimic_robotiq_hande">
         <joint>${prefix}finger_joint</joint>
-        <mimicJoint>${prefix}robotiq_hande_base_to_right_finger</mimicJoint>
+        <mimicJoint>${prefix}right_finger_joint</mimicJoint>
+        <multiplier>1.0</multiplier>
+        <offset>0.0</offset>
       </plugin>
     </gazebo>
