Commit message: Renamed robotiq_dual_coupling to robotiq_dual_bracket

File: urdf/robotiq_dual_bracket.urdf.xacro (robot description, xacro)
@@ -1,5 +1,5 @@
 <?xml version="1.0"?>
 <robot xmlns:xacro="http://ros.org/wiki/xacro">
-  <xacro:macro name="robotiq_dual_coupling" params="prefix parent *origin">
+  <xacro:macro name="robotiq_dual_bracket" params="prefix parent *origin">
     <xacro:property name="h_offset" value="0.0427"/>
     <xacro:property name="v_offset" value="0.0266"/>
@@ -13,5 +13,5 @@
         <origin xyz="-0.0685 -0.1215 0.024" rpy="${-pi/2} ${-pi/2} 0" />
         <geometry>
-          <mesh filename="package://aist_robotiq/meshes/visual/robotiq_dual_coupling.stl"
+          <mesh filename="package://aist_robotiq/meshes/visual/robotiq_dual_bracket.stl"
 		scale="0.001 0.001 0.001"/>
         </geometry>
@@ -23,5 +23,5 @@
         <origin xyz="-0.068 -0.120 0.024" rpy="${-pi/2} ${-pi/2} 0" />
         <geometry>
-          <mesh filename="package://aist_robotiq/meshes/collision/robotiq_dual_coupling.stl" />
+          <mesh filename="package://aist_robotiq/meshes/collision/robotiq_dual_bracket.stl" />
         </geometry>
       </collision>

Commit message: Fixed scale of collision model of robotiq_dual_bracket

File: urdf/robotiq_dual_bracket.urdf.xacro (robot description, xacro)
@@ -14,5 +14,5 @@
         <geometry>
           <mesh filename="package://aist_robotiq/meshes/visual/robotiq_dual_bracket.stl"
-		scale="0.001 0.001 0.001"/>
+	  	scale="0.001 0.001 0.001"/>
         </geometry>
         <material name="">
@@ -23,5 +23,6 @@
         <origin xyz="-0.068 -0.120 0.024" rpy="${-pi/2} ${-pi/2} 0" />
         <geometry>
-          <mesh filename="package://aist_robotiq/meshes/collision/robotiq_dual_bracket.stl" />
+          <mesh filename="package://aist_robotiq/meshes/collision/robotiq_dual_bracket.stl"
+	  	scale="0.001 0.001 0.001"/>
         </geometry>
       </collision>
