Commit message: Move tip_link of robotiq grippers to urdf of aist_robotiq package

File: urdf/robotiq_140_gripper.urdf.xacro (robot description, xacro)
@@ -246,4 +246,10 @@
       <origin xyz="0 0 0" rpy="${pi} ${-pi/2} 0"/>
     </joint>
+    <joint name="${prefix}tip_link_joint" type="fixed">
+      <parent link="${prefix}base_link"/>
+      <child link="${prefix}tip_link"/>
+      <origin rpy="0.0 0.0 0.0" xyz=".233 0.0 0.0"/>
+    </joint>
+    <link name="${prefix}tip_link"/>
     <xacro:robotiq_arg2f_base_link prefix="${prefix}"/>
     <xacro:finger_links prefix="${prefix}" fingerprefix="left" stroke="140"/>

File: urdf/robotiq_85_gripper.urdf.xacro (robot description, xacro)
@@ -237,4 +237,10 @@
       <origin xyz="0 0 0" rpy="${pi} ${-pi/2} 0"/>
     </joint>
+    <joint name="${prefix}tip_link_joint" type="fixed">
+      <parent link="${prefix}base_link"/>
+      <child link="${prefix}tip_link"/>
+      <origin rpy="0.0 0.0 0.0" xyz=".163 0.0 0.0"/>
+    </joint>
+    <link name="${prefix}tip_link"/>
     <xacro:robotiq_arg2f_base_link prefix="${prefix}"/>
     <xacro:finger_links prefix="${prefix}" fingerprefix="left" stroke="85"/>

File: urdf/robotiq_hande_gripper.urdf.xacro (robot description, xacro)
@@ -19,4 +19,10 @@
       <origin xyz="0 0 0" rpy="${pi/2} 0 ${pi/2}"/>
     </joint>
+    <joint name="${prefix}tip_link_joint" type="fixed">
+      <parent link="${prefix}base_link"/>
+      <child link="${prefix}tip_link"/>
+      <origin rpy="0.0 0.0 0.0" xyz=".146 0.0 0.0"/>
+    </joint>
+    <link name="${prefix}tip_link"/>
     <link name="${prefix}hande_link">
       <inertial>
