Commit message: Make nodelet only

File: urdf/PhoXi3Dscanner_macro.xacro (robot description, xacro)
@@ -1,35 +1,36 @@
 <?xml version="1.0" ?>
 <robot xmlns:xacro="http://ros.org/wiki/xacro">
-    <xacro:macro name = "PhoXi3Dscanner" params ="scanner_parent scanner_name *scanner_origin sensor_parent sensor_name *sensor_origin *visual *collision">
-        <joint name="${scanner_parent}_to_${scanner_name}_joint" type="fixed">
-            <parent link="${scanner_parent}"/>
-            <child link="${scanner_name}"/>
-            <xacro:insert_block name="scanner_origin" />
-        </joint>
-        <joint name="${sensor_parent}_to_${sensor_name}_joint" type="fixed">
-            <parent link="${sensor_parent}"/>
-            <child link="${sensor_name}"/>
-            <xacro:insert_block name="sensor_origin" />
-        </joint>
-        <link name="${scanner_name}">
-            <visual>
-                <!-- <origin xyz="0 0 0" rpy="0 1.5707 0" /> -->
-		<origin xyz="0 0 0" rpy="0 ${pi/2} ${pi}"/>
-                <geometry>
-                    <xacro:insert_block name="visual" />
-                </geometry>
-                <material name="">
-                    <color rgba="0.8 0.8 0.8 1"/>
-                </material>
-            </visual>
-            <collision>
-                <!-- <origin xyz="0 0 0" rpy="0 1.5707 0" /> -->
-		<origin xyz="0 0 0" rpy="0 ${pi/2} ${pi}"/>
-                <geometry>
-                    <xacro:insert_block name="collision" />
-                </geometry>
-            </collision>
-        </link>
-        <link name="${sensor_name}"/>
-    </xacro:macro>
+  <xacro:macro name="PhoXi3Dscanner"
+	       params="scanner_parent scanner_name *scanner_origin sensor_parent sensor_name *sensor_origin *visual *collision">
+    <joint name="${scanner_parent}_to_${scanner_name}_joint" type="fixed">
+      <parent link="${scanner_parent}"/>
+      <child  link="${scanner_name}"/>
+      <xacro:insert_block name="scanner_origin" />
+    </joint>
+    <joint name="${sensor_parent}_to_${sensor_name}_joint" type="fixed">
+      <parent link="${sensor_parent}"/>
+      <child  link="${sensor_name}"/>
+      <xacro:insert_block name="sensor_origin" />
+    </joint>
+    <link name="${scanner_name}">
+      <visual>
+        <!-- <origin xyz="0 0 0" rpy="0 1.5707 0" /> -->
+	<origin xyz="0 0 0" rpy="0 ${pi/2} ${pi}"/>
+        <geometry>
+          <xacro:insert_block name="visual" />
+        </geometry>
+        <material name="">
+          <color rgba="0.8 0.8 0.8 1"/>
+        </material>
+      </visual>
+      <collision>
+        <!-- <origin xyz="0 0 0" rpy="0 1.5707 0" /> -->
+	<origin xyz="0 0 0" rpy="0 ${pi/2} ${pi}"/>
+        <geometry>
+          <xacro:insert_block name="collision" />
+        </geometry>
+      </collision>
+    </link>
+    <link name="${sensor_name}"/>
+  </xacro:macro>
 </robot>

File: urdf/PhoXi3Dscanner_values.xacro (robot description, xacro)
@@ -1,48 +1,58 @@
 <?xml version="1.0" ?>
 <robot xmlns:xacro="http://ros.org/wiki/xacro">
-    <!--PhoXi3Dscanner XS-->
-    <xacro:macro name="PhoXi3DscannerXS_default_sensor_origin">
-        <!-- <origin xyz="0.1 0.025 0.035" rpy="0 -0.26965337 0" /> -->
-        <origin xyz="-0.1 -0.03 0.035" rpy="0 0 0" />
-    </xacro:macro>
-    <xacro:macro name="PhoXi3DscannerXS_meshes">
-        <mesh filename="package://aist_phoxi_camera/meshes/visual/PhoXi_XS.f.STL" scale = "0.001 0.001 0.001"/>
-        <mesh filename="package://aist_phoxi_camera/meshes/collision/PhoXi_XS.c.STL" scale = "0.001 0.001 0.001"/>
-    </xacro:macro>
-    <!--PhoXi3Dscanner S-->
-    <xacro:macro name="PhoXi3DscannerS_default_sensor_origin">
-        <!-- <origin xyz="${0.23 / 2.0} 0.0168 0.035" rpy="0 -0.26965337 0" /> -->
-        <origin xyz="${0.23 / 2.0} -0.03 0.035" rpy="0 -0.26965337 0" />
-    </xacro:macro>
-    <xacro:macro name="PhoXi3DscannerS_meshes">
-        <mesh filename="package://aist_phoxi_camera/meshes/visual/PhoXi_S.f.STL" scale = "0.001 0.001 0.001"/>
-        <mesh filename="package://aist_phoxi_camera/meshes/collision/PhoXi_S.c.STL" scale = "0.001 0.001 0.001"/>
-    </xacro:macro>
-    <!--PhoXi3Dscanner M-->
-    <xacro:macro name="PhoXi3DscannerM_default_sensor_origin">
-        <!-- <origin xyz="${0.350 / 2.0} 0.0168 0.035" rpy="0 -0.20507619 0" /> -->
-        <origin xyz="${0.350 / 2.0} -0.03 0.035" rpy="0 -0.20507619 0" />
-    </xacro:macro>
-    <xacro:macro name="PhoXi3DscannerM_meshes">
-        <mesh filename="package://aist_phoxi_camera/meshes/visual/PhoXi_M.f.STL" scale = "0.001 0.001 0.001"/>
-        <mesh filename="package://aist_phoxi_camera/meshes/collision/PhoXi_M.c.STL" scale = "0.001 0.001 0.001"/>
-    </xacro:macro>
-    <!--PhoXi3Dscanner L-->
-    <xacro:macro name="PhoXi3DscannerL_default_sensor_origin">
-        <!-- <origin xyz="${(0.55 / 2.0)} 0.0168 0.035" rpy="0 -0.1649336 0" /> -->
-        <origin xyz="${(0.55 / 2.0)} -0.03 0.035" rpy="0 -0.1649336 0" />
-    </xacro:macro>
-    <xacro:macro name="PhoXi3DscannerL_meshes">
-        <mesh filename="package://aist_phoxi_camera/meshes/visual/PhoXi_L.f.STL" scale = "0.001 0.001 0.001"/>
-        <mesh filename="package://aist_phoxi_camera/meshes/collision/PhoXi_L.c.STL" scale = "0.001 0.001 0.001"/>
-    </xacro:macro>
-    <!--PhoXi3Dscanner XL-->
-    <xacro:macro name="PhoXi3DscannerXL_default_sensor_origin">
-        <!-- <origin xyz="${0.850 / 2.0} 0.0168 0.035" rpy="0 -0.1309 0" /> -->
-        <origin xyz="${0.850 / 2.0} -0.03 0.035" rpy="0 -0.1309 0" />
-    </xacro:macro>
-    <xacro:macro name="PhoXi3DscannerXL_meshes">
-        <mesh filename="package://aist_phoxi_camera/meshes/visual/PhoXi_XL.f.STL" scale = "0.001 0.001 0.001"/>
-        <mesh filename="package://aist_phoxi_camera/meshes/collision/PhoXi_XL.c.STL" scale = "0.001 0.001 0.001"/>
-    </xacro:macro>
+  <!--PhoXi3Dscanner XS-->
+  <xacro:macro name="PhoXi3DscannerXS_default_sensor_origin">
+    <!-- <origin xyz="0.1 0.025 0.035" rpy="0 -0.26965337 0" /> -->
+    <origin xyz="-0.1 -0.03 0.035" rpy="0 0 0" />
+  </xacro:macro>
+  <xacro:macro name="PhoXi3DscannerXS_meshes">
+    <mesh filename="package://aist_phoxi_camera/meshes/visual/PhoXi_XS.f.STL"
+	  scale = "0.001 0.001 0.001"/>
+    <mesh filename="package://aist_phoxi_camera/meshes/collision/PhoXi_XS.c.STL"
+	  scale = "0.001 0.001 0.001"/>
+  </xacro:macro>
+  <!--PhoXi3Dscanner S-->
+  <xacro:macro name="PhoXi3DscannerS_default_sensor_origin">
+    <!-- <origin xyz="${0.23 / 2.0} 0.0168 0.035" rpy="0 -0.26965337 0" /> -->
+    <origin xyz="${0.23 / 2.0} -0.03 0.035" rpy="0 -0.26965337 0" />
+  </xacro:macro>
+  <xacro:macro name="PhoXi3DscannerS_meshes">
+    <mesh filename="package://aist_phoxi_camera/meshes/visual/PhoXi_S.f.STL"
+	  scale = "0.001 0.001 0.001"/>
+    <mesh filename="package://aist_phoxi_camera/meshes/collision/PhoXi_S.c.STL"
+	  scale = "0.001 0.001 0.001"/>
+  </xacro:macro>
+  <!--PhoXi3Dscanner M-->
+  <xacro:macro name="PhoXi3DscannerM_default_sensor_origin">
+    <!-- <origin xyz="${0.350 / 2.0} 0.0168 0.035" rpy="0 -0.20507619 0" /> -->
+    <origin xyz="${0.350 / 2.0} -0.03 0.035" rpy="0 -0.20507619 0" />
+  </xacro:macro>
+  <xacro:macro name="PhoXi3DscannerM_meshes">
+    <mesh filename="package://aist_phoxi_camera/meshes/visual/PhoXi_M.f.STL"
+	  scale = "0.001 0.001 0.001"/>
+    <mesh filename="package://aist_phoxi_camera/meshes/collision/PhoXi_M.c.STL"
+	  scale = "0.001 0.001 0.001"/>
+  </xacro:macro>
+  <!--PhoXi3Dscanner L-->
+  <xacro:macro name="PhoXi3DscannerL_default_sensor_origin">
+    <!-- <origin xyz="${(0.55 / 2.0)} 0.0168 0.035" rpy="0 -0.1649336 0" /> -->
+    <origin xyz="${(0.55 / 2.0)} -0.03 0.035" rpy="0 -0.1649336 0" />
+  </xacro:macro>
+  <xacro:macro name="PhoXi3DscannerL_meshes">
+    <mesh filename="package://aist_phoxi_camera/meshes/visual/PhoXi_L.f.STL"
+	  scale = "0.001 0.001 0.001"/>
+    <mesh filename="package://aist_phoxi_camera/meshes/collision/PhoXi_L.c.STL"
+	  scale = "0.001 0.001 0.001"/>
+  </xacro:macro>
+  <!--PhoXi3Dscanner XL-->
+  <xacro:macro name="PhoXi3DscannerXL_default_sensor_origin">
+    <!-- <origin xyz="${0.850 / 2.0} 0.0168 0.035" rpy="0 -0.1309 0" /> -->
+    <origin xyz="${0.850 / 2.0} -0.03 0.035" rpy="0 -0.1309 0" />
+  </xacro:macro>
+  <xacro:macro name="PhoXi3DscannerXL_meshes">
+    <mesh filename="package://aist_phoxi_camera/meshes/visual/PhoXi_XL.f.STL"
+	  scale = "0.001 0.001 0.001"/>
+    <mesh filename="package://aist_phoxi_camera/meshes/collision/PhoXi_XL.c.STL"
+	  scale = "0.001 0.001 0.001"/>
+  </xacro:macro>
 </robot>

File: urdf/phoxi_m_camera.urdf.xacro (robot description, xacro)
@@ -1,23 +1,17 @@
 <?xml version="1.0"?>
 <robot name="phoxi_m_camera" xmlns:xacro="http://wiki.ros.org/xacro">
-  <xacro:macro name="phoxi_m_camera" params="prefix parent *origin">
+  <xacro:macro name="phoxi_m_camera" params="name parent *origin">
     <xacro:include filename="$(find aist_phoxi_camera)/urdf/PhoXi3Dscanner_values.xacro"/>
     <xacro:include filename="$(find aist_phoxi_camera)/urdf/PhoXi3Dscanner_macro.xacro"/>
     <xacro:PhoXi3Dscanner scanner_parent="${parent}"
-			  scanner_name  ="${prefix}camera"
-			  sensor_parent ="${prefix}camera"
-			  sensor_name   ="${prefix}sensor">
+			  scanner_name  ="${name}_link"
+			  sensor_parent ="${name}_link"
+			  sensor_name   ="${name}_sensor">
       <xacro:insert_block name="origin"/>
       <xacro:PhoXi3DscannerM_default_sensor_origin/>
       <xacro:PhoXi3DscannerM_meshes/>
     </xacro:PhoXi3Dscanner>
-    <link name="${prefix}camera_link"/>
-    <joint name="${prefix}sensor_to_${prefix}camera_link" type="fixed">
-      <parent link="${prefix}sensor"/>
-      <child  link="${prefix}camera_link"/>
-      <origin xyz="0 0 0" rpy="${pi/2} ${-pi/2} 0"/>
-    </joint>
-    <gazebo reference="${prefix}camera_link">
-      <sensor name="${prefix}camera" type="depth">
+    <gazebo reference="${name}_sensor">
+      <sensor name="${name}" type="depth">
 	<always_on>true</always_on>
 	<visualize>true</visualize>
@@ -36,11 +30,11 @@
           </clip>
 	</camera>
-	<plugin name="${prefix}cam_controller"
+	<plugin name="${name}_controller"
 		filename="libgazebo_ros_openni_kinect.so">
           <baseline>0.35</baseline>
           <alwaysOn>true</alwaysOn>
           <updateRate>2.5</updateRate>
-          <cameraName>${prefix}camera</cameraName>
-          <frameName>${prefix}sensor</frameName>
+          <cameraName>${name}</cameraName>
+          <frameName>${name}_sensor</frameName>
           <imageTopicName>texture</imageTopicName>
           <depthImageTopicName>depth_map</depthImageTopicName>

Commit message: Add reference frame for gazebo

File: urdf/PhoXi3Dscanner_macro.xacro (robot description, xacro)
@@ -33,4 +33,11 @@
     </link>
     <link name="${sensor_name}"/>
+    <link name="${sensor_name}_reference"/>
+    <joint name="${sensor_name}_to_${sensor_name}_reference_joint"
+	   type="fixed">
+      <parent link="${sensor_name}"/>
+      <child  link="${sensor_name}_reference"/>
+      <origin xyz="0 0 0" rpy="${pi/2} ${-pi/2} 0"/>
+    </joint>
   </xacro:macro>
 </robot>

File: urdf/phoxi_m_camera.urdf.xacro (robot description, xacro)
@@ -12,5 +12,5 @@
       <xacro:PhoXi3DscannerM_meshes/>
     </xacro:PhoXi3Dscanner>
-    <gazebo reference="${name}_sensor">
+    <gazebo reference="${name}_sensor_reference">
       <sensor name="${name}" type="depth">
 	<always_on>true</always_on>

Commit message: Reorganize meshes and URDF of aist_phoxi_camera

File: urdf/PhoXi3Dscanner_macro.xacro (robot description, xacro)
@@ -16,5 +16,5 @@
       <visual>
         <!-- <origin xyz="0 0 0" rpy="0 1.5707 0" /> -->
-	<origin xyz="0 0 0" rpy="0 ${pi/2} ${pi}"/>
+	<origin xyz="0 0 0" rpy="0 0 0"/>
         <geometry>
           <xacro:insert_block name="visual" />
@@ -26,5 +26,5 @@
       <collision>
         <!-- <origin xyz="0 0 0" rpy="0 1.5707 0" /> -->
-	<origin xyz="0 0 0" rpy="0 ${pi/2} ${pi}"/>
+	<origin xyz="0 0 0" rpy="0 0 0"/>
         <geometry>
           <xacro:insert_block name="collision" />

File: urdf/PhoXi3Dscanner_values.xacro (robot description, xacro)
@@ -3,6 +3,6 @@
   <!--PhoXi3Dscanner XS-->
   <xacro:macro name="PhoXi3DscannerXS_default_sensor_origin">
-    <!-- <origin xyz="0.1 0.025 0.035" rpy="0 -0.26965337 0" /> -->
-    <origin xyz="-0.1 -0.03 0.035" rpy="0 0 0" />
+    <!-- <origin xyz="-0.1 -0.03 0.035" rpy="0 0 0" /> -->
+    <origin xyz="-0.090 0.03595 0.0299" rpy="${-pi/2} 0 0" />
   </xacro:macro>
   <xacro:macro name="PhoXi3DscannerXS_meshes">
@@ -14,6 +14,7 @@
   <!--PhoXi3Dscanner S-->
   <xacro:macro name="PhoXi3DscannerS_default_sensor_origin">
-    <!-- <origin xyz="${0.23 / 2.0} 0.0168 0.035" rpy="0 -0.26965337 0" /> -->
-    <origin xyz="${0.23 / 2.0} -0.03 0.035" rpy="0 -0.26965337 0" />
+    <!-- <origin xyz="${0.23 / 2.0} -0.03 0.035" rpy="0 -0.26965337 0" /> -->
+    <origin xyz="0.1173845315 0.005287752939 0.0299"
+	    rpy="${-pi/2} 0 ${15.45/180*pi}" />
   </xacro:macro>
   <xacro:macro name="PhoXi3DscannerS_meshes">
@@ -26,5 +27,6 @@
   <xacro:macro name="PhoXi3DscannerM_default_sensor_origin">
     <!-- <origin xyz="${0.350 / 2.0} 0.0168 0.035" rpy="0 -0.20507619 0" /> -->
-    <origin xyz="${0.350 / 2.0} -0.03 0.035" rpy="0 -0.20507619 0" />
+    <origin xyz="0.176277236938477 0.002164826095 0.0299"
+	    rpy="${-pi/2} 0 ${11.75/180*pi}" />
   </xacro:macro>
   <xacro:macro name="PhoXi3DscannerM_meshes">
@@ -36,6 +38,7 @@
   <!--PhoXi3Dscanner L-->
   <xacro:macro name="PhoXi3DscannerL_default_sensor_origin">
-    <!-- <origin xyz="${(0.55 / 2.0)} 0.0168 0.035" rpy="0 -0.1649336 0" /> -->
-    <origin xyz="${(0.55 / 2.0)} -0.03 0.035" rpy="0 -0.1649336 0" />
+    <!-- <origin xyz="${(0.55 / 2.0)} -0.03 0.035" rpy="0 -0.1649336 0" /> -->
+    <origin xyz="0.274213 0.0090044 0.0299"
+	    rpy="${-pi/2} 0 ${9.45/180*pi}" />
   </xacro:macro>
   <xacro:macro name="PhoXi3DscannerL_meshes">
@@ -48,5 +51,6 @@
   <xacro:macro name="PhoXi3DscannerXL_default_sensor_origin">
     <!-- <origin xyz="${0.850 / 2.0} 0.0168 0.035" rpy="0 -0.1309 0" /> -->
-    <origin xyz="${0.850 / 2.0} -0.03 0.035" rpy="0 -0.1309 0" />
+    <origin xyz="0.4349977156 0.02086702926 0.0299"
+	    rpy="${-pi/2} 0 ${7.5/180*pi}" />
   </xacro:macro>
   <xacro:macro name="PhoXi3DscannerXL_meshes">
@@ -58,10 +62,10 @@
   <!--MotionCam3D M-->
   <xacro:macro name="MotionCam3D_M_default_sensor_origin">
-    <origin xyz="${0.350 / 2.0} -0.03 0.035" rpy="0 0 0" />
+    <origin xyz="${0.350 / 2.0} 0.03 0.035" rpy="${-pi/2} 0 0" />
   </xacro:macro>
   <xacro:macro name="MotionCam3D_M_meshes">
-    <mesh filename="package://aist_phoxi_camera/meshes/visual/MotionCam3D_M.STL"
+    <mesh filename="package://aist_phoxi_camera/meshes/visual/MotionCam3D_M.f.STL"
 	  scale = "0.001 0.001 0.001"/>
-    <mesh filename="package://aist_phoxi_camera/meshes/collision/MotionCam3D_M.STL"
+    <mesh filename="package://aist_phoxi_camera/meshes/collision/MotionCam3D_M.c.STL"
 	  scale = "0.001 0.001 0.001"/>
   </xacro:macro>
