Commit message: Reorganize meshes and URDF of aist_phoxi_camera

File: urdf/PhoXi3Dscanner_macro.xacro (robot description, xacro)
@@ -2,16 +2,18 @@
 <robot xmlns:xacro="http://ros.org/wiki/xacro">
   <xacro:macro name="PhoXi3Dscanner"
-	       params="scanner_parent scanner_name *scanner_origin sensor_parent sensor_name *sensor_origin *visual *collision">
-    <joint name="${scanner_parent}_to_${scanner_name}_joint" type="fixed">
-      <parent link="${scanner_parent}"/>
-      <child  link="${scanner_name}"/>
-      <xacro:insert_block name="scanner_origin" />
+	       params="parent name image_width image_height
+		       horizontal_fov base_line update_rate
+		       *origin *reference *visual *collision">
+    <joint name="${name}_link_joint" type="fixed">
+      <parent link="${parent}"/>
+      <child  link="${name}_link"/>
+      <xacro:insert_block name="origin" />
     </joint>
-    <joint name="${sensor_parent}_to_${sensor_name}_joint" type="fixed">
-      <parent link="${sensor_parent}"/>
-      <child  link="${sensor_name}"/>
-      <xacro:insert_block name="sensor_origin" />
+    <joint name="${name}_reference_joint" type="fixed">
+      <parent link="${name}_link"/>
+      <child  link="${name}_reference"/>
+      <xacro:insert_block name="reference" />
     </joint>
-    <link name="${scanner_name}">
+    <link name="${name}_link">
       <visual>
         <!-- <origin xyz="0 0 0" rpy="0 1.5707 0" /> -->
@@ -32,12 +34,56 @@
       </collision>
     </link>
-    <link name="${sensor_name}"/>
-    <link name="${sensor_name}_reference"/>
-    <joint name="${sensor_name}_to_${sensor_name}_reference_joint"
+    <link name="${name}_reference"/>
+    <link name="${name}_sensor"/>
+    <joint name="${name}_sensor_joint"
 	   type="fixed">
-      <parent link="${sensor_name}"/>
-      <child  link="${sensor_name}_reference"/>
-      <origin xyz="0 0 0" rpy="${pi/2} ${-pi/2} 0"/>
+      <parent link="${name}_reference"/>
+      <child  link="${name}_sensor"/>
+      <origin xyz="0 0 0" rpy="${-pi/2} 0 ${-pi/2}"/>
     </joint>
+    <gazebo reference="${name}_sensor_reference">
+      <sensor name="${name}" type="depth">
+	<always_on>true</always_on>
+	<visualize>true</visualize>
+	<camera>
+          <image>
+            <width>${image_width}</width>
+            <height>${image_height}</height>
+            <format>L8</format>
+          </image>
+          <horizontal_fov>${horizontal_fov}</horizontal_fov>
+          <depth_camera>
+          </depth_camera>
+          <clip>
+            <near>0.1</near>
+            <far>100</far>
+          </clip>
+	</camera>
+	<plugin name="${name}_controller"
+		filename="libgazebo_ros_openni_kinect.so">
+          <baseline>${base_line}</baseline>
+          <alwaysOn>true</alwaysOn>
+          <updateRate>${update_rate}</updateRate>
+          <cameraName>${name}</cameraName>
+          <frameName>${name}_sensor</frameName>
+          <imageTopicName>texture</imageTopicName>
+          <depthImageTopicName>depth_map</depthImageTopicName>
+          <pointCloudTopicName>pointcloud</pointCloudTopicName>
+          <cameraInfoTopicName>camera_info</cameraInfoTopicName>
+          <depthImageCameraInfoTopicName>camera_info</depthImageCameraInfoTopicName>
+          <pointCloudCutoff>0.4</pointCloudCutoff>
+          <!-- <hackBaseline>0.35</hackBaseline> -->
+          <distortionK1>0.0</distortionK1>
+          <distortionK2>0.0</distortionK2>
+          <distortionK3>0.0</distortionK3>
+          <distortionT1>0.0</distortionT1>
+          <distortionT2>0.0</distortionT2>
+          <CxPrime>0.0</CxPrime>
+          <Cx>0.0</Cx>
+          <Cy>0.0</Cy>
+          <focalLength>0.0</focalLength>
+	</plugin>
+      </sensor>
+    </gazebo>
   </xacro:macro>
 </robot>

File: urdf/PhoXi3Dscanner_values.xacro (robot description, xacro)
@@ -2,7 +2,7 @@
 <robot xmlns:xacro="http://ros.org/wiki/xacro">
   <!--PhoXi3Dscanner XS-->
-  <xacro:macro name="PhoXi3DscannerXS_default_sensor_origin">
+  <xacro:macro name="PhoXi3DscannerXS_default_reference">
     <!-- <origin xyz="-0.1 -0.03 0.035" rpy="0 0 0" /> -->
-    <origin xyz="-0.090 0.03595 0.0299" rpy="${-pi/2} 0 0" />
+    <origin xyz="0.03595 0.090 0.0299" rpy="0 0 0" />
   </xacro:macro>
   <xacro:macro name="PhoXi3DscannerXS_meshes">
@@ -12,9 +12,14 @@
 	  scale = "0.001 0.001 0.001"/>
   </xacro:macro>
+  <xacro:property name="PhoXi3DscannerXS_image_width"	 value="2064"/>
+  <xacro:property name="PhoXi3DscannerXS_image_height"	 value="1544"/>
+  <xacro:property name="PhoXi3DscannerXS_horizontal_fov" value="0.6519"/>
+  <xacro:property name="PhoXi3DscannerXS_base_line"	 value="0.085"/>
+  <xacro:property name="PhoXi3DscannerXS_update_rate"	 value="2.5"/>
   <!--PhoXi3Dscanner S-->
-  <xacro:macro name="PhoXi3DscannerS_default_sensor_origin">
+  <xacro:macro name="PhoXi3DscannerS_default_reference">
     <!-- <origin xyz="${0.23 / 2.0} -0.03 0.035" rpy="0 -0.26965337 0" /> -->
-    <origin xyz="0.1173845315 0.005287752939 0.0299"
-	    rpy="${-pi/2} 0 ${15.45/180*pi}" />
+    <origin xyz="0.005287752939 -0.1173845315 0.0299"
+	    rpy="0 0 ${15.45/180*pi}" />
   </xacro:macro>
   <xacro:macro name="PhoXi3DscannerS_meshes">
@@ -24,9 +29,14 @@
 	  scale = "0.001 0.001 0.001"/>
   </xacro:macro>
+  <xacro:property name="PhoXi3DscannerS_image_width"	value="2064"/>
+  <xacro:property name="PhoXi3DscannerS_image_height"	value="1544"/>
+  <xacro:property name="PhoXi3DscannerS_horizontal_fov"	value="0.8145"/>
+  <xacro:property name="PhoXi3DscannerS_base_line"	value="0.23"/>
+  <xacro:property name="PhoXi3DscannerS_update_rate"	value="2.5"/>
   <!--PhoXi3Dscanner M-->
-  <xacro:macro name="PhoXi3DscannerM_default_sensor_origin">
+  <xacro:macro name="PhoXi3DscannerM_default_reference">
     <!-- <origin xyz="${0.350 / 2.0} 0.0168 0.035" rpy="0 -0.20507619 0" /> -->
-    <origin xyz="0.176277236938477 0.002164826095 0.0299"
-	    rpy="${-pi/2} 0 ${11.75/180*pi}" />
+    <origin xyz="0.002164826095 -0.176277236938477 0.0299"
+	    rpy="0 0 ${11.75/180*pi}" />
   </xacro:macro>
   <xacro:macro name="PhoXi3DscannerM_meshes">
@@ -36,9 +46,14 @@
 	  scale = "0.001 0.001 0.001"/>
   </xacro:macro>
+  <xacro:property name="PhoXi3DscannerM_image_width"	value="2064"/>
+  <xacro:property name="PhoXi3DscannerM_image_height"	value="1544"/>
+  <xacro:property name="PhoXi3DscannerM_horizontal_fov"	value="0.9077"/>
+  <xacro:property name="PhoXi3DscannerM_base_line"	value="0.35"/>
+  <xacro:property name="PhoXi3DscannerM_update_rate"	value="2.5"/>
   <!--PhoXi3Dscanner L-->
-  <xacro:macro name="PhoXi3DscannerL_default_sensor_origin">
+  <xacro:macro name="PhoXi3DscannerL_default_reference">
     <!-- <origin xyz="${(0.55 / 2.0)} -0.03 0.035" rpy="0 -0.1649336 0" /> -->
-    <origin xyz="0.274213 0.0090044 0.0299"
-	    rpy="${-pi/2} 0 ${9.45/180*pi}" />
+    <origin xyz="0.0090044 -0.274213 0.0299"
+	    rpy="0 0 ${9.45/180*pi}" />
   </xacro:macro>
   <xacro:macro name="PhoXi3DscannerL_meshes">
@@ -48,9 +63,14 @@
 	  scale = "0.001 0.001 0.001"/>
   </xacro:macro>
+  <xacro:property name="PhoXi3DscannerL_image_width"	value="2064"/>
+  <xacro:property name="PhoXi3DscannerL_image_height"	value="1544"/>
+  <xacro:property name="PhoXi3DscannerL_horizontal_fov"	value="0.8733"/>
+  <xacro:property name="PhoXi3DscannerL_base_line"	value="0.55"/>
+  <xacro:property name="PhoXi3DscannerL_update_rate"	value="2.5"/>
   <!--PhoXi3Dscanner XL-->
-  <xacro:macro name="PhoXi3DscannerXL_default_sensor_origin">
+  <xacro:macro name="PhoXi3DscannerXL_default_reference">
     <!-- <origin xyz="${0.850 / 2.0} 0.0168 0.035" rpy="0 -0.1309 0" /> -->
-    <origin xyz="0.4349977156 0.02086702926 0.0299"
-	    rpy="${-pi/2} 0 ${7.5/180*pi}" />
+    <origin xyz="0.02086702926 -0.4349977156 0.0299"
+	    rpy="0 0 ${7.5/180*pi}" />
   </xacro:macro>
   <xacro:macro name="PhoXi3DscannerXL_meshes">
@@ -60,7 +80,12 @@
 	  scale = "0.001 0.001 0.001"/>
   </xacro:macro>
+  <xacro:property name="PhoXi3DscannerXL_image_width"	 value="2064"/>
+  <xacro:property name="PhoXi3DscannerXL_image_height"	 value="1544"/>
+  <xacro:property name="PhoXi3DscannerXL_horizontal_fov" value="0.8401"/>
+  <xacro:property name="PhoXi3DscannerXL_base_line"	 value="0.85"/>
+  <xacro:property name="PhoXi3DscannerXL_update_rate"	 value="2.5"/>
   <!--MotionCam3D M-->
-  <xacro:macro name="MotionCam3D_M_default_sensor_origin">
-    <origin xyz="${0.350 / 2.0} 0.03 0.035" rpy="${-pi/2} 0 0" />
+  <xacro:macro name="MotionCam3D_M_default_reference">
+    <origin xyz="0.03 ${-0.350 / 2.0} 0.035" rpy="0 0 0" />
   </xacro:macro>
   <xacro:macro name="MotionCam3D_M_meshes">
@@ -70,3 +95,8 @@
 	  scale = "0.001 0.001 0.001"/>
   </xacro:macro>
+  <xacro:property name="MotionCam3D_M_image_width"	value="1120"/>
+  <xacro:property name="MotionCam3D_M_image_height"	value="800"/>
+  <xacro:property name="MotionCam3D_M_horizontal_fov"	value="0.9180"/>
+  <xacro:property name="MotionCam3D_M_base_line"	value="0.35"/>
+  <xacro:property name="MotionCam3D_M_update_rate"	value="20.0"/>
 </robot>

File: urdf/motioncam_m_camera.urdf.xacro (robot description, xacro)
@@ -2,58 +2,18 @@
 <robot name="motioncam_m_camera" xmlns:xacro="http://wiki.ros.org/xacro">
   <xacro:macro name="motioncam_m_camera" params="name parent *origin">
-    <xacro:include filename="$(find aist_phoxi_camera)/urdf/PhoXi3Dscanner_values.xacro"/>
-    <xacro:include filename="$(find aist_phoxi_camera)/urdf/PhoXi3Dscanner_macro.xacro"/>
-    <xacro:PhoXi3Dscanner scanner_parent="${parent}"
-			  scanner_name  ="${name}_link"
-			  sensor_parent ="${name}_link"
-			  sensor_name   ="${name}_sensor">
+    <xacro:include filename="$(find aist_phoxi_camera
+			     )/urdf/PhoXi3Dscanner_values.xacro"/>
+    <xacro:include filename="$(find aist_phoxi_camera
+			     )/urdf/PhoXi3Dscanner_macro.xacro"/>
+    <xacro:PhoXi3Dscanner parent="${parent}" name="${name}"
+			  image_width="${MotionCam3D_M_image_width}"
+			  image_height="${MotionCam3D_M_image_height}"
+			  horizontal_fov="${MotionCam3D_M_horizontal_fov}"
+			  base_line="${MotionCam3D_M_base_line}"
+			  update_rate="${MotionCam3D_M_update_rate}">
       <xacro:insert_block name="origin"/>
-      <xacro:MotionCam3D_M_default_sensor_origin/>
+      <xacro:MotionCam3D_M_default_reference/>
       <xacro:MotionCam3D_M_meshes/>
     </xacro:PhoXi3Dscanner>
-    <gazebo reference="${name}_sensor_reference">
-      <sensor name="${name}" type="depth">
-	<always_on>true</always_on>
-	<visualize>true</visualize>
-	<camera>
-          <horizontal_fov>0.876</horizontal_fov>
-          <image>
-            <width>1120</width>
-            <height>800</height>
-            <format>L8</format>
-          </image>
-          <depth_camera>
-          </depth_camera>
-          <clip>
-            <near>0.1</near>
-            <far>100</far>
-          </clip>
-	</camera>
-	<plugin name="${name}_controller"
-		filename="libgazebo_ros_openni_kinect.so">
-          <baseline>0.35</baseline>
-          <alwaysOn>true</alwaysOn>
-          <updateRate>2.5</updateRate>
-          <cameraName>${name}</cameraName>
-          <frameName>${name}_sensor</frameName>
-          <imageTopicName>texture</imageTopicName>
-          <depthImageTopicName>depth_map</depthImageTopicName>
-          <pointCloudTopicName>pointcloud</pointCloudTopicName>
-          <cameraInfoTopicName>camera_info</cameraInfoTopicName>
-          <depthImageCameraInfoTopicName>camera_info</depthImageCameraInfoTopicName>
-          <pointCloudCutoff>0.4</pointCloudCutoff>
-          <!-- <hackBaseline>0.35</hackBaseline> -->
-          <distortionK1>0.0</distortionK1>
-          <distortionK2>0.0</distortionK2>
-          <distortionK3>0.0</distortionK3>
-          <distortionT1>0.0</distortionT1>
-          <distortionT2>0.0</distortionT2>
-          <CxPrime>0.0</CxPrime>
-          <Cx>0.0</Cx>
-          <Cy>0.0</Cy>
-          <focalLength>0.0</focalLength>
-	</plugin>
-      </sensor>
-    </gazebo>
   </xacro:macro>
 </robot>

File: urdf/phoxi_m_camera.urdf.xacro (robot description, xacro)
@@ -2,58 +2,18 @@
 <robot name="phoxi_m_camera" xmlns:xacro="http://wiki.ros.org/xacro">
   <xacro:macro name="phoxi_m_camera" params="name parent *origin">
-    <xacro:include filename="$(find aist_phoxi_camera)/urdf/PhoXi3Dscanner_values.xacro"/>
-    <xacro:include filename="$(find aist_phoxi_camera)/urdf/PhoXi3Dscanner_macro.xacro"/>
-    <xacro:PhoXi3Dscanner scanner_parent="${parent}"
-			  scanner_name  ="${name}_link"
-			  sensor_parent ="${name}_link"
-			  sensor_name   ="${name}_sensor">
+    <xacro:include filename="$(find aist_phoxi_camera
+			     )/urdf/PhoXi3Dscanner_values.xacro"/>
+    <xacro:include filename="$(find aist_phoxi_camera
+			     )/urdf/PhoXi3Dscanner_macro.xacro"/>
+    <xacro:PhoXi3Dscanner parent="${parent}" name="${name}"
+			  image_width="${PhoXi3DscannerM_image_width}"
+			  image_height="${PhoXi3DscannerM_image_height}"
+			  horizontal_fov="${PhoXi3DscannerM_horizontal_fov}"
+			  base_line="${PhoXi3DscannerM_base_line}"
+			  update_rate="${PhoXi3DscannerM_update_rate}">
       <xacro:insert_block name="origin"/>
-      <xacro:PhoXi3DscannerM_default_sensor_origin/>
+      <xacro:PhoXi3DscannerM_default_reference/>
       <xacro:PhoXi3DscannerM_meshes/>
     </xacro:PhoXi3Dscanner>
-    <gazebo reference="${name}_sensor_reference">
-      <sensor name="${name}" type="depth">
-	<always_on>true</always_on>
-	<visualize>true</visualize>
-	<camera>
-          <horizontal_fov>0.876</horizontal_fov>
-          <image>
-            <width>2064</width>
-            <height>1544</height>
-            <format>L8</format>
-          </image>
-          <depth_camera>
-          </depth_camera>
-          <clip>
-            <near>0.1</near>
-            <far>100</far>
-          </clip>
-	</camera>
-	<plugin name="${name}_controller"
-		filename="libgazebo_ros_openni_kinect.so">
-          <baseline>0.35</baseline>
-          <alwaysOn>true</alwaysOn>
-          <updateRate>2.5</updateRate>
-          <cameraName>${name}</cameraName>
-          <frameName>${name}_sensor</frameName>
-          <imageTopicName>texture</imageTopicName>
-          <depthImageTopicName>depth_map</depthImageTopicName>
-          <pointCloudTopicName>pointcloud</pointCloudTopicName>
-          <cameraInfoTopicName>camera_info</cameraInfoTopicName>
-          <depthImageCameraInfoTopicName>camera_info</depthImageCameraInfoTopicName>
-          <pointCloudCutoff>0.4</pointCloudCutoff>
-          <!-- <hackBaseline>0.35</hackBaseline> -->
-          <distortionK1>0.0</distortionK1>
-          <distortionK2>0.0</distortionK2>
-          <distortionK3>0.0</distortionK3>
-          <distortionT1>0.0</distortionT1>
-          <distortionT2>0.0</distortionT2>
-          <CxPrime>0.0</CxPrime>
-          <Cx>0.0</Cx>
-          <Cy>0.0</Cy>
-          <focalLength>0.0</focalLength>
-	</plugin>
-      </sensor>
-    </gazebo>
   </xacro:macro>
 </robot>

Commit message: Remove service for saving pointcloud in ply format

File: urdf/PhoXi3Dscanner_macro.xacro (robot description, xacro)
@@ -22,5 +22,5 @@
           <xacro:insert_block name="visual" />
         </geometry>
-        <material name="">
+        <material name="Gazebo/Black">
           <color rgba="0.8 0.8 0.8 1"/>
         </material>

Commit message: Use ament_cmake_auto and add hooks for gz

File: urdf/PhoXi3Dscanner_macro.xacro (robot description, xacro)
@@ -22,6 +22,6 @@
           <xacro:insert_block name="visual" />
         </geometry>
-        <material name="Gazebo/Black">
-          <color rgba="0.1 0.1 0.1 1"/>
+        <material name="">
+          <color rgba="0 0 0 1"/>
         </material>
       </visual>
@@ -42,46 +42,38 @@
       <origin xyz="0 0 0" rpy="${-pi/2} 0 ${-pi/2}"/>
     </joint>
-    <gazebo reference="${name}_reference">
-      <sensor name="${name}" type="depth">
-	<always_on>true</always_on>
-	<visualize>true</visualize>
+    <gazebo reference="${name}_sensor">
+      <sensor type="rgbd_camera" name="${name}">
 	<camera>
+	  <!-- Color sensor's FOV(VGA): 68 deg. -->
+          <horizontal_fov>${horizontal_fov}</horizontal_fov>
           <image>
+	    <!-- VGA -->
             <width>${image_width}</width>
             <height>${image_height}</height>
             <format>L8</format>
           </image>
-          <horizontal_fov>${horizontal_fov}</horizontal_fov>
-          <depth_camera>
-          </depth_camera>
           <clip>
             <near>0.1</near>
             <far>100</far>
           </clip>
+	  <gz_frame_id>${name}_sensor</gz_frame_id>
+	  <optical_frame_id>${name}_sensor</optical_frame_id>
+	  <noise>
+	    <type>gaussian</type>
+	    <mean>0.0</mean>
+	    <stddev>0.001</stddev>
+	  </noise>
+          <distortion>
+	    <k1>0.0</k1>
+	    <k2>0.0</k2>
+	    <k3>0.0</k3>
+	    <p1>0.0</p1>
+	    <p2>0.0</p2>
+	  </distortion>
 	</camera>
-	<plugin name="${name}_controller"
-		filename="libgazebo_ros_openni_kinect.so">
-          <baseline>${base_line}</baseline>
-          <alwaysOn>true</alwaysOn>
-          <updateRate>${update_rate}</updateRate>
-          <cameraName>${name}</cameraName>
-          <frameName>${name}_sensor</frameName>
-          <imageTopicName>texture</imageTopicName>
-          <depthImageTopicName>depth_map</depthImageTopicName>
-          <pointCloudTopicName>pointcloud</pointCloudTopicName>
-          <cameraInfoTopicName>camera_info</cameraInfoTopicName>
-          <depthImageCameraInfoTopicName>camera_info</depthImageCameraInfoTopicName>
-          <pointCloudCutoff>0.4</pointCloudCutoff>
-          <!-- <hackBaseline>0.35</hackBaseline> -->
-          <distortionK1>0.0</distortionK1>
-          <distortionK2>0.0</distortionK2>
-          <distortionK3>0.0</distortionK3>
-          <distortionT1>0.0</distortionT1>
-          <distortionT2>0.0</distortionT2>
-          <CxPrime>0.0</CxPrime>
-          <Cx>0.0</Cx>
-          <Cy>0.0</Cy>
-          <focalLength>0.0</focalLength>
-	</plugin>
+	<always_on>true</always_on>
+        <updateRate>${update_rate}</updateRate>
+	<visualize>true</visualize>
+	<topic>${name}</topic>
       </sensor>
     </gazebo>
