Commit message: Intrroduce use_nominal_extrinsics parameter

File: urdf/PhoXi3Dscanner_macro.xacro (robot description, xacro)
@@ -2,5 +2,6 @@
 <robot xmlns:xacro="http://ros.org/wiki/xacro">
   <xacro:macro name="PhoXi3Dscanner"
-	       params="parent name image_width image_height
+	       params="parent name use_nominal_extrinsics
+		       image_width image_height
 		       horizontal_fov base_line update_rate
 		       *origin *reference *visual *collision">
@@ -9,9 +10,4 @@
       <child  link="${name}_link"/>
       <xacro:insert_block name="origin" />
-    </joint>
-    <joint name="${name}_reference_joint" type="fixed">
-      <parent link="${name}_link"/>
-      <child  link="${name}_reference"/>
-      <xacro:insert_block name="reference" />
     </joint>
     <link name="${name}_link">
@@ -34,48 +30,55 @@
       </collision>
     </link>
-    <link name="${name}_reference"/>
-    <link name="${name}_sensor"/>
-    <joint name="${name}_sensor_joint"
-	   type="fixed">
-      <parent link="${name}_reference"/>
-      <child  link="${name}_sensor"/>
-      <origin xyz="0 0 0" rpy="${-pi/2} 0 ${-pi/2}"/>
-    </joint>
-    <gazebo reference="${name}_reference">
-      <sensor type="rgbd_camera" name="${name}">
-	<camera>
-	  <!-- Color sensor's FOV(VGA): 68 deg. -->
-          <horizontal_fov>${horizontal_fov}</horizontal_fov>
-          <image>
-	    <!-- VGA -->
-            <width>${image_width}</width>
-            <height>${image_height}</height>
-            <format>L8</format>
-          </image>
-          <clip>
-            <near>0.1</near>
-            <far>100</far>
-          </clip>
-	  <frame_id>${name}_reference</frame_id>
-	  <optical_frame_id>${name}_sensor</optical_frame_id>
-	  <noise>
-	    <type>gaussian</type>
-	    <mean>0.0</mean>
-	    <stddev>0.001</stddev>
-	  </noise>
-          <distortion>
-	    <k1>0.0</k1>
-	    <k2>0.0</k2>
-	    <k3>0.0</k3>
-	    <p1>0.0</p1>
-	    <p2>0.0</p2>
-	  </distortion>
-	</camera>
-	<always_on>true</always_on>
-        <updateRate>${update_rate}</updateRate>
-	<visualize>true</visualize>
-	<topic>${name}</topic>
-      </sensor>
-    </gazebo>
+    <xacro:if value="${use_nominal_extrinsics}">
+      <link name="${name}_reference"/>
+      <joint name="${name}_reference_joint" type="fixed">
+	<parent link="${name}_link"/>
+	<child  link="${name}_reference"/>
+	<xacro:insert_block name="reference" />
+      </joint>
+      <link name="${name}_sensor"/>
+      <joint name="${name}_sensor_joint"
+	     type="fixed">
+	<parent link="${name}_reference"/>
+	<child  link="${name}_sensor"/>
+	<origin xyz="0 0 0" rpy="${-pi/2} 0 ${-pi/2}"/>
+      </joint>
+      <gazebo reference="${name}_reference">
+	<sensor type="rgbd_camera" name="${name}">
+	  <camera>
+	    <!-- Color sensor's FOV(VGA): 68 deg. -->
+            <horizontal_fov>${horizontal_fov}</horizontal_fov>
+            <image>
+	      <!-- VGA -->
+              <width>${image_width}</width>
+              <height>${image_height}</height>
+              <format>L8</format>
+            </image>
+            <clip>
+              <near>0.1</near>
+              <far>100</far>
+            </clip>
+	    <frame_id>${name}_reference</frame_id>
+	    <optical_frame_id>${name}_sensor</optical_frame_id>
+	    <noise>
+	      <type>gaussian</type>
+	      <mean>0.0</mean>
+	      <stddev>0.001</stddev>
+	    </noise>
+            <distortion>
+	      <k1>0.0</k1>
+	      <k2>0.0</k2>
+	      <k3>0.0</k3>
+	      <p1>0.0</p1>
+	      <p2>0.0</p2>
+	    </distortion>
+	  </camera>
+	  <always_on>true</always_on>
+          <updateRate>${update_rate}</updateRate>
+	  <visualize>true</visualize>
+	  <topic>${name}</topic>
+	</sensor>
+      </gazebo>
+    </xacro:if>
   </xacro:macro>
 </robot>

File: urdf/motioncam_m_camera.urdf.xacro (robot description, xacro)
@@ -1,5 +1,6 @@
 <?xml version="1.0"?>
 <robot name="motioncam_m_camera" xmlns:xacro="http://wiki.ros.org/xacro">
-  <xacro:macro name="motioncam_m_camera" params="name parent *origin">
+  <xacro:macro name="motioncam_m_camera"
+	       params="name parent use_nominal_extrinsics *origin">
     <xacro:include filename="$(find aist_phoxi_camera
 			     )/urdf/PhoXi3Dscanner_values.xacro"/>
@@ -7,4 +8,5 @@
 			     )/urdf/PhoXi3Dscanner_macro.xacro"/>
     <xacro:PhoXi3Dscanner parent="${parent}" name="${name}"
+			  use_nominal_extrinsics="${use_nominal_extrinsics}"
 			  image_width="${MotionCam3D_M_image_width}"
 			  image_height="${MotionCam3D_M_image_height}"

File: urdf/phoxi_l_camera.urdf.xacro (robot description, xacro)
@@ -1,5 +1,6 @@
 <?xml version="1.0"?>
 <robot name="phoxi_l_camera" xmlns:xacro="http://wiki.ros.org/xacro">
-  <xacro:macro name="phoxi_l_camera" params="name parent *origin">
+  <xacro:macro name="phoxi_l_camera"
+	       params="name parent use_nominal_extrinsics:=false *origin">
     <xacro:include filename="$(find aist_phoxi_camera
 			     )/urdf/PhoXi3Dscanner_values.xacro"/>
@@ -7,4 +8,5 @@
 			     )/urdf/PhoXi3Dscanner_macro.xacro"/>
     <xacro:PhoXi3Dscanner parent="${parent}" name="${name}"
+			  use_nominal_extrinsics="${use_nominal_extrinsics}"
 			  image_width="${PhoXi3DscannerL_image_width}"
 			  image_height="${PhoXi3DscannerL_image_height}"

File: urdf/phoxi_m_camera.urdf.xacro (robot description, xacro)
@@ -1,5 +1,6 @@
 <?xml version="1.0"?>
 <robot name="phoxi_m_camera" xmlns:xacro="http://wiki.ros.org/xacro">
-  <xacro:macro name="phoxi_m_camera" params="name parent *origin">
+  <xacro:macro name="phoxi_m_camera"
+	       params="name parent use_nominal_extrinsics:=false *origin">
     <xacro:include filename="$(find aist_phoxi_camera
 			     )/urdf/PhoXi3Dscanner_values.xacro"/>
@@ -7,4 +8,5 @@
 			     )/urdf/PhoXi3Dscanner_macro.xacro"/>
     <xacro:PhoXi3Dscanner parent="${parent}" name="${name}"
+			  use_nominal_extrinsics="${use_nominal_extrinsics}"
 			  image_width="${PhoXi3DscannerM_image_width}"
 			  image_height="${PhoXi3DscannerM_image_height}"

File: urdf/phoxi_s_camera.urdf.xacro (robot description, xacro)
@@ -1,5 +1,6 @@
 <?xml version="1.0"?>
 <robot name="phoxi_s_camera" xmlns:xacro="http://wiki.ros.org/xacro">
-  <xacro:macro name="phoxi_s_camera" params="name parent *origin">
+  <xacro:macro name="phoxi_s_camera"
+	       params="name parent use_nominal_extrinsics:=false *origin">
     <xacro:include filename="$(find aist_phoxi_camera
 			     )/urdf/PhoXi3Dscanner_values.xacro"/>
@@ -7,4 +8,5 @@
 			     )/urdf/PhoXi3Dscanner_macro.xacro"/>
     <xacro:PhoXi3Dscanner parent="${parent}" name="${name}"
+			  use_nominal_extrinsics="${use_nominal_extrinsics}"
 			  image_width="${PhoXi3DscannerS_image_width}"
 			  image_height="${PhoXi3DscannerS_image_height}"

File: urdf/phoxi_xl_camera.urdf.xacro (robot description, xacro)
@@ -1,5 +1,6 @@
 <?xml version="1.0"?>
 <robot name="phoxi_xl_camera" xmlns:xacro="http://wiki.ros.org/xacro">
-  <xacro:macro name="phoxi_xl_camera" params="name parent *origin">
+  <xacro:macro name="phoxi_xl_camera"
+	       params="name parent use_nominal_extrinsics:=false *origin">
     <xacro:include filename="$(find aist_phoxi_camera
 			     )/urdf/PhoXi3Dscanner_values.xacro"/>
@@ -7,4 +8,5 @@
 			     )/urdf/PhoXi3Dscanner_macro.xacro"/>
     <xacro:PhoXi3Dscanner parent="${parent}" name="${name}"
+			  use_nominal_extrinsics="${use_nominal_extrinsics}"
 			  image_width="${PhoXi3DscannerXL_image_width}"
 			  image_height="${PhoXi3DscannerXL_image_height}"

File: urdf/phoxi_xs_camera.urdf.xacro (robot description, xacro)
@@ -1,5 +1,6 @@
 <?xml version="1.0"?>
 <robot name="phoxi_xs_camera" xmlns:xacro="http://wiki.ros.org/xacro">
-  <xacro:macro name="phoxi_xs_camera" params="name parent *origin">
+  <xacro:macro name="phoxi_xs_camera"
+	       params="name parent use_nominal_extrinsics:=false *origin">
     <xacro:include filename="$(find aist_phoxi_camera
 			     )/urdf/PhoXi3Dscanner_values.xacro"/>
@@ -7,4 +8,5 @@
 			     )/urdf/PhoXi3Dscanner_macro.xacro"/>
     <xacro:PhoXi3Dscanner parent="${parent}" name="${name}"
+			  use_nominal_extrinsics="${use_nominal_extrinsics}"
 			  image_width="${PhoXi3DscannerXS_image_width}"
 			  image_height="${PhoXi3DscannerXS_image_height}"
